File: cad_files/mm9a.sch (KiCad schematic (older format))
At the start: 51 parts, among them K1 Electromagnetic_Actor, K1C1 auxcontalt, K1C2 auxcontalt, K2 Electromagnetic_Actor, K2C1 auxcontalt, K2C2 auxcontalt, K3 Electromagnetic_Actor, K3C1 auxcontalt, K3C2 auxcontalt, K4 Electromagnetic_Actor, K4C1 auxcontalt, K4C2 auxcontalt, K5 toff=10s, K5C1 auxcontalt, K6 Electromagnetic_Actor, K6C1 auxcontalt, K6C2 auxcontalt, K7 Electromagnetic_Actor, K7C1 auxcontalt, K7C2 auxcontalt, P1 screw_conn, P10 screw_conn, P11 screw_conn, P12 screw_conn, P13 screw_conn, P14 screw_conn, P15 screw_conn, P16 screw_conn, P17 screw_conn, P18 screw_conn, P19 screw_conn, P2 screw_conn, P20 screw_conn, P21 screw_conn, P22 screw_conn, P3 screw_conn, P4 screw_conn, P5 screw_conn, P6 screw_conn, P7 screw_conn, P8 screw_conn, P9 screw_conn

Commit message: 220116
Parts:
- removed K4C2: auxcontalt, symbol auxcontalt
- F1, F2, F3: value 500 mA T -> ? mA T
- F4: value fuse -> ? mA T
- F5: value 500 mA T -> 50 mA T
- F6: value 500mA T -> 400mA
- Tr1: value 230/24V 50VA -> 230/24V 8VA
Connections:
- net at K1.1 (-), K2.1 (-), K3.1 (-)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: no longer P11.1, P13.1, P9.1
- net at K2C1.~ (B): now also K1C1.~ (B), K3C1.~ (B), K6C1.~ (B), PS2.~ (B)
- net at K2C2.~ (B): now also F2.1
- net at K1C2.~ (B): now also F1.1
- net at K4C1.~ (B): now also F4.1
- net at P6.1, Tr1.~: now also P11.1, P13.1, P21.1, P9.1; no longer K4C1.~ (B)
- net at F5.2, P5.1: now also K1C2.~ (B), K2C2.~ (B), K3C2.~ (B), K4C1.~ (B)
- net at K3C2.~ (B): now also F3.1
- net at PS2.~ (B): now also K6.2 (+)
- net at K6C1.~ (B): now also K5.1 (-), K5C1.~ (B), K7C1.~ (B), PS1.~ (B)
- net at PS1.~ (B): now also K5C1.~ (B), K7.2 (+)
- new net: F6.1, K1C1.~ (B), K2C1.~ (B), K3C1.~ (B), P4.1
- new net: F6.2, Tr1.~
- now unconnected: K1C1.~ (B), K1C1.~ (B), K3C1.~ (B), K3C1.~ (B), K5C1.~ (B), K5C1.~ (B), K7C1.~ (B)
- no-connect marks 13 -> 12
Other:
- note added: "Common 24V AC"
- note added: "Control input #1"
- note added: "Control input #2"
- note added: "Control input #3"
- note added: "Electromagnetic\n valve out #1\n\n 230V AC"
- note added: "Electromagnetic\n valve out #2\n\n 230V AC"
- note added: "Electromagnetic\n valve out #3\n\n 230V AC"
- note added: "Main voltage input\n230V 50-60Hz"
- note added: "Water pump out\n\n 230V AC"
- note removed: "24V AC"
- note removed: "Control input"
- note removed: "Electromagnetic\nvalve out #1"
- note removed: "Electromagnetic\nvalve out #2"
- note removed: "Electromagnetic\nvalve out #3"
- note removed: "IN1"
- note removed: "IN2"
- note removed: "IN3"
- note removed: "L1"
- note removed: "L2"
- note removed: "Main voltage input\n230 V 50-60 Hz"
- note removed: "Water pump out"
- moved on the sheet: F1, F2, F3, F4, F5, F6, K1, K1C1, K1C2, K2, K2C1, K2C2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

Commit message: 220203
Parts:
- removed F4: ? mA T, symbol fuse
- removed F5: 50 mA T, symbol fuse
- added P21, P22, P23: screw_conn, symbol screw_conn
- P1, P11, P14, P17, P18, P19, P2, P20, P3, P4, P5, P8: Color (none) -> gray
- P10, P13, P16, P7: Color (none) -> green/yellow
- P12, P15, P6, P9: Color (none) -> blue
- P24: renamed from P21; Color (none) -> blue
- P25: renamed from P22; Color (none) -> green/yellow
- renumbered F6 to F1, F1 to F2, F2 to F3, F3 to F4, K4 to K1, K4C1 to K1C1, K1 to K2, K1C1 to K2C1, K1C2 to K2C2, K2 to K3, K2C1 to K3C1, K2C2 to K3C2, K3 to K4, K3C1 to K4C1, K3C2 to K4C2, K7 to K6, K7C1 to K6C1, K7C2 to K6C2, K6 to K7, K6C1 to K7C1, K6C2 to K7C2
Connections:
- net at K3C1.~ (B): now also K2C1.~ (B), K4C1.~ (B), K7C1.~ (B), PS2.~ (B)
- net at K3C2.~ (B): now also F3.1
- net at K2C2.~ (B): now also F2.1
- net at K1C1.~ (B): now also P23.1
- net at K4C2.~ (B): now also F4.1
- net at F4.2: now also P14.1; no longer P12.1
- net at F3.2: now also P11.1; no longer P10.1
- net at P20.1: now also K6C2.~ (B)
- net at Tr1.~: now also P12.1, P15.1, P24.1, P6.1, P9.1
- net at P25.1, P7.1: now also P10.1, P13.1, P16.1
- net at PS2.~ (B): now also K7.2 (+)
- net at K7C1.~ (B): now also K5.1 (-), K5C1.~ (B), K6C1.~ (B), PS1.~ (B)
- net at PS1.~ (B): now also K5C1.~ (B), K6.2 (+)
- net at K6C2.~ (B): now also P22.1; no longer P17.1
- net at P18.1: now also K7C2.~ (B); no longer K6C2.~ (B)
- net at P19.1: now also K7C2.~ (B); no longer K6C2.~ (B)
- new net: F1.1, K2C1.~ (B), K3C1.~ (B), K4C1.~ (B), P4.1
- new net: K1C1.~ (B), K2C2.~ (B), K3C2.~ (B), K4C2.~ (B), P5.1, Tr1.~
- new net: K6C2.~ (B), P21.1
- new net: K7C2.~ (B), P17.1
- now unconnected: K2C1.~ (B), K2C1.~ (B), K4C1.~ (B), K4C1.~ (B), K5C1.~ (B), K5C1.~ (B), K6C1.~ (B)

Commit message: 220404
Parts:
- removed P10, P12, P13, P16, P19, P21, P22, P9: screw_conn, symbol screw_conn
- removed Tr1: 230/24V 8VA, symbol transformer_1P_1S
- added D1, D2, D3, D4, D5, D6: 1N4001, symbol D
- added F4: 500 mA T, symbol fuse
- added U1-1, U1-2, U1-3, U1-4: screw_conn, symbol screw_conn
- F1: renamed from F2; value ? mA T -> 500 mA T
- F2: renamed from F3; value ? mA T -> 500 mA T
- F3: renamed from F4; value ? mA T -> 500 mA T
- F5: renamed from F1; value 400mA -> 500 mA
- K7: renamed from K5; value toff=10s -> toff=5s
- renumbered K2 to K1, K2C1 to K1C1, K2C2 to K1C2, K3 to K2, K3C1 to K2C1, K3C2 to K2C2, K4 to K3, K4C1 to K3C1, K4C2 to K3C2, K1 to K4, K1C1 to K4C1, K7 to K5, K7C1 to K5C1, K7C2 to K5C2, K5C1 to K7C1, P11 to P10, P14 to P11, P17 to P12, P18 to P13, P20 to P14, P23 to P15, P24 to P16, P25 to P17, P15 to P8, P8 to P9
Connections:
- net at K1.1 (-), K2.1 (-), K3.1 (-)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: now also P8.1, D1.2 (A), D2.2 (A), D3.2 (A), D4.2 (A), D5.2 (A), D6.2 (A), U1-4.1
- net at K2.2 (+), P2.1: now also D2.1 (K)
- net at K2C1.~ (B): now also K1C1.~ (B), K3C1.~ (B), K5C1.~ (B), PS2.~ (B)
- net at K2C2.~ (B): now also F2.1
- net at K1.2 (+), P1.1: now also D1.1 (K)
- net at K1C2.~ (B): now also F1.1
- net at K4.2 (+), K6C1.~ (B): now also D4.1 (K)
- net at K4C1.~ (B): now also P15.1
- net at K3.2 (+), P3.1: now also D3.1 (K)
- net at K3C2.~ (B): now also F3.1
- net at F5.2: now also K1C2.~ (B), K2C2.~ (B), K3C2.~ (B), U1-3.1
- net at P16.1, P6.1: now also U1-2.1; no longer P8.1
- net at PS2.~ (B): now also K5.2 (+), D5.1 (K)
- net at K5C1.~ (B): now also K6C1.~ (B), K7.1 (-), K7C1.~ (B), PS1.~ (B)
- net at PS1.~ (B): now also K6.2 (+), K7C1.~ (B), D6.1 (K)
- net at K6C2.~ (B), P14.1: now also K5C2.~ (B)
- net at K6C2.~ (B): now also P13.1
- new net: F5.1, K1C1.~ (B), K2C1.~ (B), K3C1.~ (B), P4.1
- new net: F4.2, K4C1.~ (B), P5.1
- new net: F4.1, U1-1.1
- now unconnected: K1C1.~ (B), K1C1.~ (B), K3C1.~ (B), K3C1.~ (B), K6C1.~ (B), K7C1.~ (B), K7C1.~ (B)
- no-connect marks 12 -> 14
Other:
- note added: "+24V - Valve #1 output"
- note added: "+24V - Valve #2 output"
- note added: "+24V - Valve #3 output"
- note added: "-24 V"
- note added: "24V DC 2A\n\nPower supply\n\n 230V AC\n"
- note added: "<Pmin"
- note added: ">Pmax"
- note added: "Common"
- note added: "L 230V AC - Water pump output"
- note added: "Main voltage input\n230 V AC"
- note added: "U1"
- note removed: "C"
- note removed: "Electromagnetic\n valve out #1\n\n 230V AC"
- note removed: "Electromagnetic\n valve out #2\n\n 230V AC"
- note removed: "Electromagnetic\n valve out #3\n\n 230V AC"
- note removed: "Main voltage input\n230V 50-60Hz"
- note removed: "NC"
- note removed: "NO"
- note removed: "Pressure error:\n P < Pmin"
- note removed: "Pressure error:\n P > Pmax"
- note removed: "Water pump out\n\n 230V AC"
- moved on the sheet: F1, F2, F3, F5, K7, K7C1, P11, P12, P13, P14, P8, P9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

Commit message: 220413
Parts:
- removed D1, D2, D3, D4, D5, D6: 1N4001, symbol D
- removed F1, F2, F3: 500 mA T, symbol fuse
- removed U1-1, U1-2, U1-3, U1-4: screw_conn, symbol screw_conn
- added D1: 100V 3A, symbol D_Bridge_+-AA
- added K4C2: auxcontalt, symbol auxcontalt
- added Trs1: 230/24V 50VA, symbol transformer_1P_1S
- F1: renamed from F4; value 500 mA T -> 0.3A T
- F2: renamed from F5; value 500 mA -> 2A
- K1, K2, K3, K4, K5, K6: value Electromagnetic_Actor -> RM84-2012-35-1024
- K7: value toff=5s -> ERV-03D
- renumbered P7 to P1, P6 to P2, P5 to P3, P1 to P5, P2 to P6, P3 to P7
Connections:
- net -24V: now reaches K1.1 (-), K2.1 (-), K3.1 (-), K4.1 (-), K5.1 (-), K6.1 (-), K7.2 (+), P8.1
- net -24V: now also D1.2 (-)
- net +24V: now reaches K2C1.~ (B)
- net +24V: now also K1C1.~ (B), K1C2.~ (B), K2C2.~ (B), K3C1.~ (B), K3C2.~ (B), P4.1, D1.1 (+)
- net at K4C1.~ (B): now also P15.1
- net at P9.1: now also K1C2.~ (B)
- net at P10.1: now also K2C2.~ (B)
- net at P11.1: now also K3C2.~ (B)
- net at P16.1: now also K4C2.~ (B); no longer P2.1
- net at PS2.~ (B): now also K5.2 (+)
- net at K5C1.~ (B): now also K6C1.~ (B), K7.1 (-), K7C1.~ (B), PS1.~ (B)
- net at PS1.~ (B): now also K6.2 (+), K7C1.~ (B)
- net at K6C2.~ (B): now also P13.1
- net at K5C2.~ (B): now also P12.1
- net at F1.1: now also Trs1.~
- new net: K1C1.~ (B), K2C1.~ (B), K3C1.~ (B), K5C1.~ (B), PS2.~ (B)
- new net: K4C1.~ (B), P3.1, Trs1.~
- new net: D1.3, F2.1
- new net: F2.2, Trs1.~
- new net: K5C2.~ (B), K6C2.~ (B), P14.1
- new net: F1.2, K4C2.~ (B), P2.1
- new net: D1.4, Trs1.~
- now unconnected: K6C1.~ (B), K7C1.~ (B), K7C1.~ (B)
- no-connect marks 14 -> 15
Other:
- note added: "Main voltage input\n 230 V AC"
- note added: "Water pump output\n 230V AC"
- note added: "low\nnormal"
- note added: "normal\nhigh"
- note removed: "24V DC 2A\n\nPower supply\n\n 230V AC\n"
- note removed: "L 230V AC - Water pump output"
- note removed: "Main voltage input\n230 V AC"
- note removed: "U1"
- moved on the sheet: F1, F2, K1, K1C1, K1C2, K2, K2C1, K2C2, K3, K3C1, K3C2, K4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

Commit message: 220425
Parts:
- removed PS1: pmin, symbol auxcontalt
- removed PS2: pmax, symbol auxcontalt
- added P10, P11, P8, P9: screw_conn, symbol screw_conn
- D1-4: renamed from D1; value 100V 3A -> 4x1N5408
- renumbered K7 to K6, K7C1 to K6C1, K6 to K7, K6C1 to K7C1, K6C2 to K7C2, P13 to P12, P12 to P13, P8 to P15, P9 to P16, P10 to P17, P11 to P18, P15 to P19, P16 to P20, P17 to P21
Connections:
- net at K4C1.~ (B): now also P19.1
- net at K5.2 (+): now also P11.1
- net at K5C1.~ (B): now also K6.1 (-), K6C1.~ (B), K7C1.~ (B), P9.1
- net at K6C1.~ (B), K7.2 (+): now also P8.1
- net at K7C2.~ (B): now also P12.1
- net at K5C2.~ (B): now also P13.1
- new net: K1C1.~ (B), K2C1.~ (B), K3C1.~ (B), K5C1.~ (B), P10.1
- new net: K4C1.~ (B), P3.1, Trs1.~
- new net: K5C2.~ (B), K7C2.~ (B), P14.1
- now unconnected: K6C1.~ (B), K7C1.~ (B)
- no-connect marks 15 -> 13
Other:
- note added: "#1"
- note added: "#2"
- note added: "#3"
- note added: "<Pmin\npressure sensor\n"
- note added: ">Pmax\npressure sensor\n"
- note added: "Control input\n\n 24V DC"
- note added: "Error output"
- note added: "Main voltage input\n\n 230 V AC"
- note added: "Valve output\n\n 24V DC"
- note added: "Water pump output\n\n 230V AC"
- note added: "common"
- note removed: "+24V - Valve #1 output"
- note removed: "+24V - Valve #2 output"
- note removed: "+24V - Valve #3 output"
- note removed: "-24 V"
- note removed: "Common"
- note removed: "Common 24V AC"
- note removed: "Control input #1"
- note removed: "Control input #2"
- note removed: "Control input #3"
- note removed: "Main voltage input\n 230 V AC"
- note removed: "Water pump output\n 230V AC"
- note removed: "low\nnormal"
- note removed: "normal\nhigh"
- moved on the sheet: K4, K4C1, K4C2, K5C1, K5C2, P1, P12, P13, P14, P19, P2, P20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

Commit message: 220512
Parts:
- F1: value 0.3A T -> 0.4A T
- K6: value ERV-03D -> timer 5s
Connections:
- net at K4C1.~ (B): now also P19.1
- net at K5C1.~ (B): now also K6.1 (-), K6C1.~ (B), K7C1.~ (B), P9.1
- net at K7C2.~ (B): now also P12.1
- net at K5C2.~ (B): now also P13.1
- net -24V: no longer names the net of D1-4.2 (-), K1.1 (-), K2.1 (-), K3.1 (-), K4.1 (-), K5.1 (-), K6.2 (+), K7.1 (-), P15.1
- new net: K1C1.~ (B), K2C1.~ (B), K3C1.~ (B), K5C1.~ (B), P10.1
- new net: K4C1.~ (B), P3.1, Trs1.~
- new net: K5C2.~ (B), K7C2.~ (B), P14.1
- now unconnected: K6C1.~ (B), K7C1.~ (B)
Other:
- note added: "+24V"
- note added: "CI1"
- note added: "CI2"
- note added: "CI3"
- note added: "Control inputs\n"
- note added: "E-COM"
- note added: "E-PMN"
- note added: "E-PMX"
- note added: "Error outputs"
- note added: "GND"
- note added: "S-PMN"
- note added: "S-PMX"
- note added: "VO1"
- note added: "VO2"
- note added: "VO3"
- note added: "Valve outputs\n\n 24V DC"
- note added: "WPO-L"
- note added: "WPO-N"
- note added: "WPO-PE"
- note removed: "#1"
- note removed: "#2"
- note removed: "#3"
- note removed: "<Pmin"
- note removed: ">Pmax"
- note removed: "Control input\n\n 24V DC"
- note removed: "Error output"
- note removed: "Valve output\n\n 24V DC"
- note removed: "common"
Changed lines of the file:
@@
 $EndComp
 Text Notes 9200 5740 0    50   ~ 0
-L
+WPO-L
 $Comp
 L screw_conn P16
@@
 $EndComp
 Text Notes 9200 2040 0    50   ~ 0
-common
+GND
 Text Notes 9200 2240 0    50   ~ 0
-#1
+VO1
 $Comp
 L screw_conn P20
@@
 $EndComp
 Text Notes 9200 5540 0    50   ~ 0
-N
+WPO-N
 $Comp
 L screw_conn P21
@@
 $EndComp
 Text Notes 9200 5950 0    50   ~ 0
-PE
+WPO-PE
 $Comp
 L Electromagnetic_Actor K5
@@
 P 5200 4800
 F 0 "K6" H 5050 5000 50  0000 L CNN
-F 1 "ERV-03D" H 5050 4500 50  0000 L CNN
+F 1 "timer 5s" H 5050 4500 50  0000 L CNN
 F 2 "" V 5175 4900 50  0000 C CNN
 F 3 "" V 5175 4900 50  0000 C CNN
@@
 NoConn ~ 6350 4900
 Text Notes 9200 4140 0    50   ~ 0
-<Pmin
+E-PMN
 Text Notes 9200 3940 0    50   ~ 0
->Pmax
+E-PMX
 Text Notes 2350 1380 2    50   ~ 0
-#1
+CI1
 $Comp
 L screw_conn P1
@@
 	-1   0    0    1
 $EndComp
-Text Notes 2475 1175 2    50   ~ 0
-common
+Text Notes 2350 1175 2    50   ~ 0
++24V
 Text Notes 2350 5530 2    50   ~ 0
 N
@@
 Main voltage input\n\n  230 V AC
 Text Notes 2350 1575 2    50   ~ 0
-#2
+CI2
 Text Notes 2350 1775 2    50   ~ 0
-#3
+CI3
 $Comp
 L screw_conn P6
@@
 P 4200 5050
 F 0 "F1" V 4300 5050 50  0000 C CNN
-F 1 "0.3A T" V 4100 5050 50  0000 C CNN
+F 1 "0.4A T" V 4100 5050 50  0000 C CNN
 F 2 "" V 4130 5050 50  0001 C CNN
 F 3 "" H 4200 5050 50  0001 C CNN
@@
 NoConn ~ 5800 3750
 Text Notes 9200 4325 0    50   ~ 0
-common
+E-COM
 Text Notes 9200 2425 0    50   ~ 0
-#2
+VO2
 Text Notes 9200 2625 0    50   ~ 0
-#3
+VO3
 $Comp
 L transformer_1P_1S Trs1
@@
 Text Label 4000 2550 1    60   ~ 0
 +24V
-Text Label 4800 3250 1    60   ~ 0
--24V
 Wire Wire Line
 	4200 4750 4200 4900
 Wire Wire Line
 	4200 5200 4200 5700
-Text Notes 9375 5825 0    50   ~ 0
+Text Notes 9550 5825 0    50   ~ 0
 Water pump output\n\n      230V AC
-Text Notes 2100 1650 2    50   ~ 0
-Control input\n\n    24V DC
-Text Notes 9875 2500 2    50   ~ 0
-Valve output\n\n    24V DC
-Text Notes 10075 4150 2    50   ~ 0
-Error output
+Text Notes 9625 2475 0    50   ~ 0
+Valve outputs\n\n   24V DC
+Text Notes 10145 4140 2    50   ~ 0
+Error outputs
 $Comp
 L screw_conn P10
@@
 Wire Wire Line
 	8450 3100 8750 3100
-Text Notes 9200 3075 0    50   ~ 0
+Text Notes 9625 3050 0    50   ~ 0
    >Pmax\npressure sensor\n
 Wire Wire Line
@@
 Connection ~ 6000 1900
 Connection ~ 6000 1300
-Text Notes 9175 3575 0    50   ~ 0
+Text Notes 9625 3550 0    50   ~ 0
    <Pmin\npressure sensor\n
+Text Notes 2075 1475 2    50   ~ 0
+Control inputs\n
+Text Notes 9200 2925 0    50   ~ 0
+S-PMX
+Text Notes 9200 3125 0    50   ~ 0
+S-PMX
+Text Notes 9175 3425 0    50   ~ 0
+S-PMN
+Text Notes 9175 3625 0    50   ~ 0
+S-PMN
 $EndSCHEMATC
